Commit message: Intent de robot dissenyat amb urdf

File: urdf/piatek.urdf (robot description, URDF)
Before this commit: robot physics, 16 links, 15 joints
Links:
- removed link box
- removed link gripper_pole
- removed link head
- removed link left_back_wheel
- removed link left_base
- removed link left_front_wheel
- removed link left_gripper
- removed link left_leg
- removed link left_tip
- removed link right_back_wheel
- removed link right_base
- removed link right_front_wheel
- removed link right_gripper
- removed link right_leg
- removed link right_tip
- added link camera_link; visual box size=0.05 0.05 0.02
- added link left_wheel_link, mass 1; collision cylinder length=0.05 radius=0.075; visual cylinder length=0.05 radius=0.075
- added link right_wheel_link, mass 1; collision cylinder length=0.05 radius=0.075; visual cylinder length=0.05 radius=0.075
- added link upper_base_link; visual cylinder length=0.30 radius=0.085
- link base_link: mass 10 -> None; geometry visual box size=0.32 0.26 0.085
Joints:
- removed joint base_to_left_leg
- removed joint base_to_right_leg
- removed joint gripper_extension
- removed joint head_swivel
- removed joint left_back_wheel_joint
- removed joint left_base_joint
- removed joint left_front_wheel_joint
- removed joint left_gripper_joint
- removed joint left_tip_joint
- removed joint right_back_wheel_joint
- removed joint right_base_joint
- removed joint right_front_wheel_joint
- removed joint right_gripper_joint
- removed joint right_tip_joint
- removed joint tobox
- added joint base_to_upper_base_joint: type fixed, parent base_link, child upper_base_link, origin xyz=0 0 0 rpy=0 0 0
- added joint left_wheel_joint: type continuous, parent base_link, child left_wheel_link, origin xyz=0.133333333333 0 -0.085 rpy=0 0 0, axis 1 0 0
- added joint right_wheel_joint: type continuous, parent base_link, child right_wheel_link, origin xyz=0.133333333333 0 -0.085 rpy=0 0 0, axis 1 0 0
- added joint upper_base_to_camera_joint: type revolute, parent upper_base_link, child camera_link, origin xyz=0 0 0 rpy=0 0 0, axis 0 0 1, limit lower=-3.1416 upper=3.1416 effort=10 velocity=3
